Commit message: youbot: remove arm for tutorial purposes

File: robots/youbot.urdf.xacro (robot description, xacro)
@@ -13,7 +13,7 @@
   <xacro:include filename="$(find youbot_description)/urdf/youbot_plate/plate.urdf.xacro" />
   <!-- youbot arm -->
-  <xacro:include filename="$(find youbot_description)/urdf/youbot_arm/arm.urdf.xacro"/>
+  <!--xacro:include filename="$(find youbot_description)/urdf/youbot_arm/arm.urdf.xacro"/-->
   <!-- youbot gripper -->
-  <xacro:include filename="$(find youbot_description)/urdf/youbot_gripper/gripper.urdf.xacro" />
+  <!--xacro:include filename="$(find youbot_description)/urdf/youbot_gripper/gripper.urdf.xacro" /-->
   <!-- controller manager -->
   <xacro:include filename="$(find youbot_description)/controller/ros_controller.urdf.xacro" />
@@ -42,5 +42,5 @@
   </xacro:youbot_gripper>
   <!-- base laser front -->
-  <xacro:hokuyo_urg04_laser name="base_laser_front" parent="base" ros_topic="base_scan" update_rate="10" min_angle="-1.57" max_angle="1.57">
+  <xacro:hokuyo_urg04_laser name="base_laser_front" parent="base" ros_topic="scan_front" update_rate="10" min_angle="-1.57" max_angle="1.57">
     <origin xyz="0.3 0 -0.03" rpy="0 0 0"/>
   </xacro:hokuyo_urg04_laser>

File: urdf/youbot_arm/arm.urdf.xacro (robot description, xacro)
@@ -6,5 +6,5 @@
 	<xacro:include filename="$(find youbot_description)/urdf/youbot_arm/arm.gazebo.xacro" />
 	<xacro:include filename="$(find youbot_description)/urdf/youbot_arm/arm.transmission.xacro" />
-        <xacro:include filename="$(find youbot_description)/urdf/youbot_arm/limits.urdf.xacro" />
+	<xacro:include filename="$(find youbot_description)/urdf/youbot_arm/limits.urdf.xacro" />
 	<xacro:macro name="youbot_arm" params="parent name *origin">
 		<!-- joint between base_link and arm_0_link -->
@@ -26,5 +26,5 @@
 					<mesh filename="package://youbot_description/meshes/youbot_arm/arm0.dae" />
 				</geometry>
-				<material name="DarkGrey" />
+				<material name="youBot/DarkGrey" />
 			</visual>
 			<collision>
@@ -37,178 +37,6 @@
 			</collision>
 		</link>
-		<!-- joint between arm_0_link and arm_1_link -->
-		<joint name="${name}_joint_1" type="revolute">
-			<origin xyz="0.024 0 0.096" rpy="0 0 ${170 * M_PI / 180}"/>
-			<parent link="${name}_link_0"/>
-			<child link="${name}_link_1"/>
-			<axis xyz="0 0 -1"/>
-			<!--<calibration rising="${arm_1_ref}" falling="${arm_1_ref}"/>-->
-			<dynamics damping="1" friction="1" />
-			<!-- damping - N*s/m, N*s*m/rad -->
-			<!-- friction - N, N*m -->
-			<limit effort="${9.5}" velocity="${M_PI / 2.0}" lower="0" upper="${joint_1_limit}"/>
-			<!--effort - N, N*m-->
-			<!--velocity - m/s, rad/s-->
-			<safety_controller k_position="20" k_velocity="${9.5/M_PI / 2.0}" soft_lower_limit="${threshold}" soft_upper_limit="${joint_1_limit_soft}" />
-			<!--k_position N/m, N/rad-->
-			<!--k_velocity N*s/m, N*s*m/rad-->
-			<!--for details: http://www.ros.org/wiki/pr2_controller_manager/safety_limits-->
-		</joint>
-		<link name="${name}_link_1">
-			<inertial>
-				<mass value="${link_1_mass}"/>
-				<xacro:link_1_inertia_tensor />
-			</inertial>
-			<visual>
-				<origin xyz="0 0 0" rpy="0 0 0" />
-				<geometry>
-					<mesh filename="package://youbot_description/meshes/youbot_arm/arm1.dae" />
-				</geometry>
-				<!--<material name="Orange" />-->
-			</visual>
-			<collision>
-				<!--<origin xyz="0 0 -0.003" rpy="0 0 0" />-->
-				<origin xyz="0 0 0" rpy="0 0 0" />
-				<geometry>
-					<mesh filename="package://youbot_description/meshes/youbot_arm/arm1_convex.dae" />
-					<!--<cylinder length="0.102" radius="0.080"/>-->
-				</geometry>
-			</collision>
-		</link>
-		<!-- joint between arm_1_link and arm_2_link -->
-		<joint name="${name}_joint_2" type="revolute">
-			<origin xyz="0.033 0 0.019" rpy="0 ${-65 * M_PI / 180} 0"/>
-			<parent link="${name}_link_1"/>
-			<child link="${name}_link_2"/>
-			<axis xyz="0 1 0"/>
-			<!--<calibration rising="${arm_2_ref}" falling="${arm_2_ref}"/>-->
-			<dynamics damping="1" friction="1" />
-			<limit effort="${9.5}" velocity="${M_PI / 2.0}" lower="0" upper="${joint_2_limit}"/>
-                        <safety_controller k_position="20" k_velocity="${2*9.5/M_PI}" soft_lower_limit="${threshold}" soft_upper_limit="${joint_2_limit_soft}" />
-		</joint>
-		<link name="${name}_link_2">
-			<inertial>
-				<mass value="${link_2_mass}"/>
-				<xacro:link_2_inertia_tensor />
-			</inertial>
-			<visual>
-			<origin xyz="0 -0.032 0.078" rpy="0 0 0" />
-				<geometry>
-					<mesh filename="package://youbot_description/meshes/youbot_arm/arm2.dae" />
-				</geometry>
-				<material name="Orange" />
-			</visual>
-			<collision>
-				<!--<origin xyz="0.001 -0.041 0.074" rpy="0 0 0" />-->
-				<origin xyz="0 -0.032 0.078" rpy="0 0 0" />
-				<geometry>
-					<mesh filename="package://youbot_description/meshes/youbot_arm/arm2_convex.dae" />
-					<!--<box size="0.074 0.082 0.222"/>-->
-				</geometry>
-			</collision>
-		</link>
-		<!-- joint between arm_2_link and arm_3_link -->
-		<!--<joint name="${name}_joint_3" type="revolute">
-			<origin xyz="0.000 0.000 0.155" rpy="0 ${146 * M_PI / 180} 0"/>
-			<parent link="${name}_link_2"/>
-			<child link="${name}_link_3"/>
-			<axis xyz="0 1 0"/>
-			<dynamics damping="1" friction="1" />
-			<limit effort="${6}" velocity="${M_PI / 2.0}" lower="-${joint_3_limit}" upper="0"/>
-                        <safety_controller k_position="20" k_velocity="50" soft_lower_limit="-${joint_3_limit_soft}" soft_upper_limit="${threshold}" />
-		</joint>-->
-		<joint name="${name}_joint_3" type="revolute">
-			<origin xyz="0.000 0.000 0.155" rpy="0 ${146 * M_PI / 180} 0"/>
-			<parent link="${name}_link_2"/>
-			<child link="${name}_link_3"/>
-			<axis xyz="0 1 0"/>
-			<dynamics damping="1" friction="1" />
-			<limit effort="${6}" velocity="${M_PI / 2.0}" lower="-${joint_3_limit}" upper="0"/>
-                        <safety_controller k_position="20" k_velocity="50" soft_lower_limit="-${joint_3_limit_soft}" soft_upper_limit="-${threshold}" />
-		</joint>
-		<link name="${name}_link_3">
-			<inertial>
-				<mass value="${link_3_mass}"/>
-				<xacro:link_3_inertia_tensor />
-			</inertial>
-			<visual>
-				<origin xyz="0.000 0.028 0.079" rpy="0 0 0" />
-				<geometry>
-					<mesh filename="package://youbot_description/meshes/youbot_arm/arm3.dae" />
-				</geometry>
-				<material name="Orange" />
-			</visual>
-			<collision>
-				<!--<origin xyz="0.000 0.025 0.067" rpy="0 0 0" />-->
-				<origin xyz="0.000 0.028 0.079" rpy="0 0 0" />
-				<geometry>
-					<mesh filename="package://youbot_description/meshes/youbot_arm/arm3_convex.dae" />
-					<!--<box size="0.064 0.054 0.192"/>-->
-				</geometry>
-			</collision>
-		</link>
-		<!-- joint between arm_3_link and arm_4_link -->
-		<joint name="${name}_joint_4" type="revolute">
-			<origin xyz="0.000 0.000 0.135" rpy="0 ${-102.5 * M_PI / 180} 0" />
-			<parent link="${name}_link_3"/>
-			<child link="${name}_link_4"/>
-			<axis xyz="0 1 0" />
-			<!--<calibration rising="${arm_4_ref}" falling="${arm_4_ref}"/>-->
-			<dynamics damping="1" friction="1" />
-			<limit effort="${2}" velocity="${M_PI / 2.0}" lower="0" upper="${joint_4_limit}"/>
-			<safety_controller k_position="20" k_velocity="100" soft_lower_limit="0" soft_upper_limit="${joint_4_limit_soft}" />
-		</joint>
-		<link name="${name}_link_4">
-			<inertial>
-				<mass value="${link_4_mass}"/>
-				<xacro:link_4_inertia_tensor />
-			</inertial>
-			<visual>
-				<origin xyz="0 -0.010 0.029" rpy="0 0 0"/>
-				<geometry>
-					<mesh filename="package://youbot_description/meshes/youbot_arm/arm4.dae" />
-				</geometry>
-				<material name="Orange" />
-			</visual>
-			<collision>
-				<!--<origin xyz="0 0 0.026" rpy="0 0 0" />-->
-				<origin xyz="0 -0.010 0.029" rpy="0 0 0"/>
-				<geometry>
-					<mesh filename="package://youbot_description/meshes/youbot_arm/arm4_convex.dae" />
-					<!--<box size="0.058 0.100 0.118"/>-->
-				</geometry>
-			</collision>
-		</link>
-		<!-- joint between arm_4_link and arm_5_link -->
-		<joint name="${name}_joint_5" type="revolute">
-			<origin xyz="-0.002 0 0.130" rpy="0 0 ${167.5 * M_PI / 180}" />
-			<parent link="${name}_link_4"/>
-			<child link="${name}_link_5"/>
-			<axis xyz="0 0 -1" />
-			<!--<calibration rising="${arm_5_ref}" falling="${arm_5_ref}"/>-->
-			<dynamics damping="1" friction="1" />
-			<limit effort="1" velocity="${M_PI / 2.0}" lower="0" upper="${joint_5_limit}" />
-                        <safety_controller k_position="20" k_velocity="100" soft_lower_limit="0" soft_upper_limit="${joint_5_limit_soft}" />
-		</joint>
-		<link name="${name}_link_5">
-			<inertial>
-				<mass value="${link_5_mass}"/>
-				<xacro:link_5_inertia_tensor />
-			</inertial>
-			<visual>
-				<origin xyz="0.003 0 -0.034" rpy="0 0 0" />
-				<geometry>
-					<mesh filename="package://youbot_description/meshes/youbot_arm/arm5.dae" />
-				</geometry>
-				<material name="DarkGrey" />
-			</visual>
-			<collision>
-				<origin xyz="0.003 0 -0.034" rpy="0 0 0" />
-				<geometry>
-					<mesh filename="package://youbot_description/meshes/youbot_arm/arm5_convex.dae" />
-					<!--<box size="0.054 0.096 0.030"/>-->
-				</geometry>
-			</collision>
-		</link>
+		<!-- INSERT YOUR JOINTS HERE -->
+		<!-- INSERT YOUR LINKS HERE -->
 		<!-- extensions -->
 		<xacro:youbot_arm_gazebo name="${name}" />
